File: eagle/cd32_riser.brd (EAGLE design)
At the start: 124.5 x 60 mm, 37 parts, among them CN1 CD32-EXPANSION, CN2 CD32-EXPANSION, IC1 LM1117MPX-3.3, U1 STM32F10XRXT6, X1 PN87520-S

Commit message: Added punt pullup
Parts:
- added R1: (no value), rcl:M1206
- renumbered XC9572XL(BUS) to XC9572XL
Connections:
- removed net -: BT1.2
- net GND: now also BT1.2
- net PUNT_IN: now also R1.1
- net VCC: now also R1.2
Routing:
- net PUNT_IN: track 62.9 -> 66.9 mm
- net VCC: track 26.5 -> 28.1 mm, vias 1 -> 2

Commit message: Added missing 10k resistor
Parts:
- added R4: 10k, rcl:M0805
Connections:
- new net N$4: LED2.A, R4.2
- net VCC: now also R4.1
Routing:
- net VCC: track 28.1 -> 31.7 mm
- net N$4: track 0.00 -> 2.80 mm
Changed lines of the file:
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@@
 <attribute name="SPICEPREFIX" value="R" x="72.65349375" y="20.299159375" size="1.778" layer="27" rot="R180" display="off"/>
+</element>
+<element name="R4" library="rcl" library_urn="urn:adsk.eagle:library:334" package="M0805" package3d_urn="urn:adsk.eagle:package:23556/1" value="10k" x="34.12914375" y="56.674603125" rot="R90">
+<attribute name="SPICEPREFIX" value="R" x="34.12914375" y="56.674603125" size="1.778" layer="27" rot="R90" display="off"/>
 </element>
 </elements>
@@
 <wire x1="71.241609375" y1="20.31104375" x2="69.443440625" y2="20.31104375" width="0.1524" layer="1"/>
 <via x="69.443440625" y="20.31104375" extent="1-16" drill="0.35"/>
+<contactref element="R4" pad="1"/>
+<wire x1="37.59375625" y1="55.43475625" x2="34.418990625" y2="55.43475625" width="0.4064" layer="1"/>
+<wire x1="34.418990625" y1="55.43475625" x2="34.12914375" y2="55.724603125" width="0.4064" layer="1"/>
 </signal>
 <signal name="+12V">
@@
 <wire x1="30.8567125" y1="27.2905375" x2="30.8567125" y2="29.0275125" width="0.1524" layer="1"/>
 </signal>
+<signal name="N$4">
+<contactref element="R4" pad="2"/>
+<contactref element="LED2" pad="A"/>
+<wire x1="31.3506875" y1="57.67931875" x2="34.074428125" y2="57.67931875" width="0.1524" layer="1"/>
+<wire x1="34.074428125" y1="57.67931875" x2="34.12914375" y2="57.624603125" width="0.1524" layer="1"/>
+</signal>
 </signals>

Commit message: Added missing 10k resistor
Parts:
- added D1: BAT54, diode:SOT23
- added R5: 10k, rcl:M0805
Connections:
- removed net +: BT1.1
- new net N$5: BT1.1, D1.1, R5.2
- net VCC33: now also D1.3, R5.1
Routing:
- net VCC33: track 61.7 -> 104.8 mm
- net N$5: track 0.00 -> 39.6 mm
Changed lines of the file:
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@@
 </element>
 <element name="C11" library="eagle-ltspice" library_urn="urn:adsk.eagle:library:217" package="C0603" package3d_urn="urn:adsk.eagle:package:13262/1" value="22p" x="48.629109375" y="49.23508125" rot="R90">
-<attribute name="NAME" x="50.359109375" y="49.96508125" size="0.508" layer="25" ratio="15" rot="R90"/>
+<attribute name="NAME" x="47.64288125" y="38.635196875" size="0.508" layer="25" ratio="15" rot="R90"/>
 <attribute name="SPICEMODEL" value="NONE" x="48.629109375" y="49.23508125" size="1.778" layer="27" rot="R90" display="off"/>
 <attribute name="SPICEPREFIX" value="C" x="48.629109375" y="49.23508125" size="1.778" layer="27" rot="R90" display="off"/>
@@
 <attribute name="SPICEPREFIX" value="R" x="34.12914375" y="56.674603125" size="1.778" layer="27" rot="R90" display="off"/>
 </element>
+<element name="R5" library="rcl" library_urn="urn:adsk.eagle:library:334" package="M0805" package3d_urn="urn:adsk.eagle:package:23556/1" value="10k" x="86.298909375" y="56.531271875" rot="R90">
+<attribute name="SPICEPREFIX" value="R" x="86.298909375" y="56.531271875" size="1.778" layer="27" rot="R90" display="off"/>
+</element>
+<element name="D1" library="diode" library_urn="urn:adsk.eagle:library:210" package="SOT23" package3d_urn="urn:adsk.eagle:package:43389/2" value="BAT54" x="53.299728125" y="47.616975" rot="R180"/>
 </elements>
 <signals>
@@
 <wire x1="17.619115625" y1="54.8576" x2="17.674390625" y2="54.912875" width="0.3048" layer="1"/>
 <wire x1="17.674390625" y1="54.912875" x2="19.2484375" y2="54.912875" width="0.3048" layer="1"/>
+<contactref element="R5" pad="1"/>
+<contactref element="D1" pad="3"/>
+<wire x1="53.299728125" y1="46.516975" x2="52.83289375" y2="46.050140625" width="0.4064" layer="1"/>
+<wire x1="52.83289375" y1="46.050140625" x2="52.83289375" y2="40.404784375" width="0.4064" layer="1"/>
+<wire x1="86.298909375" y1="55.55111875" x2="86.298909375" y2="55.581271875" width="0.4064" layer="1"/>
+<wire x1="53.299728125" y1="46.516975" x2="61.433025" y2="46.516975" width="0.4064" layer="1"/>
+<wire x1="61.433025" y1="46.516975" x2="70.46716875" y2="55.55111875" width="0.4064" layer="1"/>
+<wire x1="70.46716875" y1="55.55111875" x2="86.298909375" y2="55.55111875" width="0.4064" layer="1"/>
 </signal>
 <signal name="TCK">
@@
 <wire x1="28.826015625" y1="23.183509375" x2="28.826015625" y2="29.0104375" width="0.1524" layer="1"/>
 </signal>
-<signal name="+">
-<contactref element="BT1" pad="1"/>
-</signal>
 <signal name="UART5_RX">
 <contactref element="U1" pad="54"/>
@@
 <wire x1="34.074428125" y1="57.67931875" x2="34.12914375" y2="57.624603125" width="0.1524" layer="1"/>
 </signal>
+<signal name="N$5">
+<contactref element="R5" pad="2"/>
+<contactref element="D1" pad="1"/>
+<contactref element="BT1" pad="1"/>
+<wire x1="54.249728125" y1="48.716975" x2="63.014025" y2="57.481271875" width="0.4064" layer="1"/>
+<wire x1="63.014025" y1="57.481271875" x2="86.298909375" y2="57.481271875" width="0.4064" layer="1"/>
+<wire x1="54.249728125" y1="48.716975" x2="54.322115625" y2="48.6445875" width="0.4064" layer="1"/>
+<wire x1="54.322115625" y1="48.6445875" x2="58.161784375" y2="48.6445875" width="0.4064" layer="1"/>
+</signal>
 </signals>

Commit message: decoupling for the CPLD.
Parts:
- added C17, C18, C19, C20, C21: (no value), rcl:C0603
Connections:
- net GND: now also C17.2, C18.2, C19.2, C20.2, C21.2
- net VCC33: now also C17.1, C18.1, C19.1, C20.1, C21.1
Routing:
- net GND: track 56.4 -> 65.8 mm, vias 24 -> 27
- net VCC33: track 104.8 -> 108.6 mm, vias 23 -> 27
