File: eagle/cd32_riser.brd (EAGLE design)
At the start: 124.5 x 60 mm, 46 parts, among them CN1 CD32-EXPANSION, CN2 CD32-EXPANSION, IC1 LM1117MPX-3.3, U1 STM32F10XRXT6, X1 PN87520-S

Commit message: updated the arm side of stuff significantly
Parts:
- removed BT1: (no value), SparkFun-Batteries:BATTCOM_20MM_PTH
- removed Q1: (no value), crystal:HC49/S
- removed SJ1, SJ2, SJ3, SJ4: (no value), jumper:SJ_2
- removed U1: STM32F10XRXT6, stm32:TQFP64
- removed X1: PN87520-S, con-berg:PN87520-S
- added G1: CH23-1220LF, battery:CH23-1220LF
- added JP1: (no value), SparkFun-Retired:1X02
- added U$1: USB-A-2_USB_USB-A-2, board:USB-A-2_USB_USB-A-2
- added U2: STM32F722RET6, STM32F722RET6:QFP50P1200X1200X160-64N
- added Y1: SMD-CRYSTAL-8MHZ-20PF-20PPM(2P-5.0X3.2MM), SMD-CRYSTAL-8MHZ-20PF-20PPM_2P-5.0X3.2MM_:X2-SMD-5.0X3.2X1.3MM
- moved JP2 79.4 mm to (119.6, 55.4), turned to 180 degrees
- moved R2 72.3 mm to (119.5, 50.7)
- moved BOOT0 31.7 mm to (84.3, 53.5)
- moved R5 31.0 mm to (57.9, 44.1), turned to 180 degrees
- moved PA9BOOT 28.5 mm to (84.3, 56.7), turned to 180 degrees
- moved R4 11.8 mm to (22.4, 57.3), flipped to the bottom, turned to 270 degrees
- moved LED1 9.22 mm to (17.8, 57.2), turned to 90 degrees
- moved LED2 8.96 mm to (22.4, 57.4), turned to 270 degrees
- moved D1 8.30 mm to (58.0, 40.8), turned to 270 degrees
- moved C3 5.75 mm to (30.1, 57.0), flipped to the top, turned to 0 degrees
- moved C2 4.03 mm to (40.1, 41.3)
- moved R3 3.74 mm to (17.8, 57.4), flipped to the bottom, turned to 90 degrees
- moved C8 3.11 mm to (39.0, 53.7), turned to 0 degrees
- moved C12 2.24 mm to (40.0, 39.1), flipped to the top, turned to 0 degrees
- moved C15 2.12 mm to (19.0, 41.5), turned to 180 degrees
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Connections:
- removed net N$1: C10.1, Q1.2, U1.5
- removed net N$10: SJ3.2, U1.38
- removed net N$11: SJ2.2, U1.39
- removed net N$2: C11.1, Q1.1, U1.6
- removed net N$3: BOOT0.2, U1.60
- removed net N$6: SJ1.2, U1.40
- removed net N$8: LED2.C, U1.29
- removed net N$9: SJ4.2, U1.37
- removed net SPI_NSS: U1.50, XC9572XL.24
- removed net USB_DM: U1.44, X1.2
- removed net USB_DP: U1.45, X1.3
- new net BOOT: BOOT0.2, U2.60
- new net INTSIG0: U2.61, XC9572XL.22
- new net INTSIG1: U2.62, XC9572XL.20
- new net INTSIG2: U2.33, XC9572XL.23
- new net INTSIG3: U2.50, XC9572XL.24
- new net INTSIG4: U2.39, XC9572XL.13
- new net INTSIG5: U2.40, XC9572XL.12
- new net INTSIG6: U2.51, XC9572XL.11
- new net INTSIG7: U2.52, XC9572XL.10
- new net INTSIG8: U2.2, XC9572XL.17
- new net LED: LED2.C, U2.29
- new net OSCIN: C10.1, U2.5, Y1.2
- new net OSCOUT: C11.1, U2.6, Y1.1
- new net USB1_DM: U$1.2-2, U2.44
- new net USB1_DP: U$1.2-3, U2.45
- new net USB2_DM: U$1.1-2, U2.35
- new net USB2_DP: U$1.1-3, U2.36
- new net VCAP_1: U2.30
- net AB: no longer U$3.P$5
- net AB_EXT: now also U$3.P$5
- net AG: no longer U$3.P$4
- net AG_EXT: now also U$3.P$4
- net AR: no longer U$3.P$3
- net AR_EXT: now also U$3.P$3
- net D24: now also U2.25
- net D25: now also U2.26
- net D26: now also U2.27
- net D27: now also U2.55
- net D28: now also U2.56
- net D29: now also U2.57
- net D30: now also U2.58
- net D31: now also U2.59
- net DKWE: now also U2.22
- net GND: now also G1.-, U$1.1-4, U$1.2-4, U$1.SHIELD1, U$1.SHIELD2, U$1.SHIELD3, U$1.SHIELD4, U2.12, U2.18, U2.31, U2.47, U2.63; no longer BT1.2, SJ1.1, SJ2.1, SJ3.1, SJ4.1, U1.12, U1.16, U1.18, U1.28, U1.31, U1.47, U1.63, X1.4
- net N$5: now also G1.+; no longer BT1.1
- net NRST: now also U2.7; no longer U1.7
- net PA9BOOT: now also U2.42; no longer U1.42
- net PUNT_IN: now also XC9572XL.9; no longer XC9572XL.13
- net PUNT_OUT: now also XC9572XL.8; no longer XC9572XL.10
- net R_W: now also U2.3, XC9572XL.5; no longer XC9572XL.7
- net SIZ0: no longer XC9572XL.4
- net SIZ1: no longer XC9572XL.2
- net SPI_CK: now also U2.8, XC9572XL.19; no longer U1.55, XC9572XL.20
- net SPI_MISO: now also U2.10, XC9572XL.18; no longer U1.56, XC9572XL.19
- net SPI_MOSI: now also U2.11, XC9572XL.16; no longer U1.57, XC9572XL.18
- net SWCLK: now also U2.49; no longer U1.49
- net SWDIO: now also U2.46; no longer U1.46
- net UART5_RX: now also JP1.1, U2.54; no longer U1.54, XC9572XL.22
- net UART5_TX: now also JP1.2, U2.53; no longer U1.53, XC9572XL.23
- net VCC: now also U$1.1-1, U$1.2-1; no longer X1.1
- net VCC33: now also U2.1, U2.13, U2.19, U2.32, U2.48, U2.64; no longer SJ1.3, SJ2.3, SJ3.3, SJ4.3, U1.1, U1.13, U1.19, U1.32, U1.48, U1.64
- net _AS: now also XC9572XL.2; no longer XC9572XL.5
- net _DKRD: now also U2.23
- net _DKWD: now also U2.41
- net _DS: now also XC9572XL.4; no longer XC9572XL.6
- net _DSACK_0: now also U2.4, XC9572XL.7; no longer XC9572XL.9
- net _DSACK_1: now also XC9572XL.6; no longer XC9572XL.8
- net _FIRE0: now also U2.20
- net _FIRE1: now also U2.21
- net _KB_CLOCK: now also U2.28; no longer XC9572XL.11
- net _KB_DATA: now also U2.9; no longer XC9572XL.12
- net _RXD: now also U2.14; no longer XC9572XL.16
- net _TXD: now also U2.15; no longer XC9572XL.17
Routing:
- net SWCLK: track 28.8 -> 116.1 mm
- net SWDIO: track 25.7 -> 112.7 mm, vias 0 -> 1
- net BOOT: track 0.00 -> 86.3 mm, vias 0 -> 1
- net _DKWD: track 27.5 -> 109.9 mm, vias 0 -> 2
- net NRST: track 26.5 -> 103.5 mm
- net _DKRD: track 27.4 -> 100.2 mm, vias 0 -> 2
- net DKWE: track 27.4 -> 100.0 mm, vias 0 -> 1
- net _FIRE0: track 27.5 -> 97.4 mm, vias 0 -> 1
- net _FIRE1: track 27.4 -> 93.8 mm, vias 0 -> 1
- net INTSIG5: track 0.00 -> 50.3 mm, vias 0 -> 2
- net INTSIG4: track 0.00 -> 50.3 mm, vias 0 -> 2
- net SIZ1: track 69.3 -> 27.4 mm
- net INTSIG8: track 0.00 -> 38.2 mm
- net R_W: track 71.4 -> 109.1 mm
- net SIZ0: track 64.6 -> 27.5 mm
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Other:
- board text added: "Terrible Fire USB CD32 Adaptor (C) 2020 S.J Leary Revision 1 Published Under the GNU GPLv2"
- board text added: "USB Circuit Derived from HID2AMI v1.1.0 https://github.com/EmberHeavyIndustries/HID2AMI"
- board text removed: "Terrible Fire USB CD32 Adaptor (C) 2020 S.J Leary Revision 0 Published Under the GNU GPLv2"
- board text removed: "USB Circuit Based on HID2AMI v1.1.0 DeLuxe by EmberHeavyIndustres 2019 https://github.com/EmberHeavyIndustries/HID2AMI"

Commit message: updated the circuit and added fuses
Parts:
- added F1, F2: 1206L050YR, 1206L050YR:FUSC3216X75N
- moved C7 14.1 mm to (42.9, 57.2), flipped to the top
- moved D1 5.64 mm to (53.6, 44.3)
- moved R5 5.64 mm to (53.5, 47.7)
- moved C3 0.39 mm to (30.5, 57.0)
- moved C8 0.11 mm to (39.0, 53.8)
Connections:
- net INTSIG0 renamed BUS_INT
- net SPI_MISO renamed SPI2_MISO
- removed net SPI_CK: U2.8, XC9572XL.19
- removed net SPI_MOSI: U2.11, XC9572XL.16
- new net N$1: F1.2, U$1.2-1
- new net N$2: F2.2, U$1.1-1
- new net SPI2_CK: U2.28, XC9572XL.19
- new net SPI2_MOSI: U2.9, XC9572XL.16
- net DKWE: now also U2.16; no longer U2.22
- net LED: now also U2.34; no longer U2.29
- net VCC: now also F1.1, F2.1; no longer U$1.1-1, U$1.2-1
- net _FIRE0: now also U2.17; no longer U2.20
- net _FIRE1: now also U2.8; no longer U2.21
- net _KB_CLOCK: now also U2.29; no longer U2.28
- net _KB_DATA: now also U2.11; no longer U2.9
Routing:
- net SPI_MOSI: track 47.7 -> 0.00 mm, vias 2 -> 0
- net SPI2_MOSI: track 0.00 -> 45.5 mm, vias 0 -> 2
- net SPI2_CK: track 0.00 -> 38.9 mm, vias 0 -> 2
- net SPI_CK: track 32.1 -> 0.00 mm, vias 2 -> 0
- net _RXD: track 90.7 -> 98.9 mm
- net DKWE: track 100.0 -> 92.3 mm
- net _KB_DATA: track 90.8 -> 83.3 mm
- net N$1: track 0.00 -> 6.57 mm
- net _KB_CLOCK: track 105.7 -> 112.0 mm
- net N$5: track 13.1 -> 18.9 mm
- net VGND: track 68.8 -> 73.8 mm
- net _FIRE1: track 93.8 -> 90.3 mm, vias 1 -> 0
- net N$2: track 0.00 -> 3.37 mm
- net UART5_RX: track 26.5 -> 29.7 mm
- net LED: track 9.46 -> 12.4 mm
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
Commit message: added the address lines
Parts:
- moved U$3 1.49 mm to (117.7, 43.9)
- moved C18 0.85 mm to (34.1, 18.8)
- moved C21 0.49 mm to (14.6, 24.9), flipped to the top
Connections:
- net A0: now also U2.24
- net A1: now also U2.37
- net A2: now also U2.38
- net INTSIG8: now also XC9572XL.18; no longer XC9572XL.17
- net SPI2_CK: now also XC9572XL.16; no longer XC9572XL.19
- net SPI2_MISO: now also XC9572XL.19; no longer XC9572XL.18
- net SPI2_MOSI: now also XC9572XL.17; no longer XC9572XL.16
Routing:
- net A1: track 30.6 -> 53.6 mm, vias 1 -> 2
- net A2: track 29.3 -> 48.1 mm, vias 1 -> 2
- net A0: track 31.4 -> 49.9 mm, vias 1 -> 2
- net SPI2_CK: track 38.9 -> 45.1 mm
- net BOOT: track 85.6 -> 89.5 mm
- net PA9BOOT: track 74.3 -> 77.2 mm
- net _HSYNC: track 54.8 -> 57.4 mm
- net _VSYNC: track 50.4 -> 52.9 mm
- net INTSIG2: track 34.4 -> 36.6 mm
- net _DKWD: track 111.7 -> 113.7 mm
- net +12V: track 98.4 -> 100.3 mm
- net INTSIG5: track 47.7 -> 45.8 mm
- net SPI2_MOSI: track 45.5 -> 43.7 mm
- net INTSIG4: track 47.6 -> 46.0 mm
- net AB_EXT: track 44.1 -> 45.7 mm
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Other:
- board text added: "GND"
- board text added: "SWCLK"
- board text added: "SWDIO"

Commit message: finished the route
Parts:
- removed LED1: (no value), led:SML0805
- added DAC: JUMPER-3PTH, SparkFun-Retired:1X03
- added PWR: (no value), led:SML0805
- added RN1, RN2: (no value), resistor-dil:CAY16
- moved C7 4.27 mm to (45.1, 53.6), turned to 180 degrees
- moved R4 3.23 mm to (19.4, 58.5), flipped to the top, turned to 0 degrees
- moved G1 1.89 mm to (71.9, 45.5)
- moved R3 1.88 mm to (19.3, 56.2), flipped to the top, turned to 180 degrees
- moved LED2 0.74 mm to (23.2, 57.4), turned to 90 degrees
- moved C11 0.71 mm to (48.7, 48.5)
- moved C6 0.62 mm to (39.0, 51.0)
- moved C8 0.37 mm to (39.1, 53.4)
- moved R5 0.34 mm to (53.6, 48.0)
Connections:
- new net AB_OUT: RN1.7, RN2.7, U$3.P$5
- new net AG_OUT: RN1.6, RN2.6, U$3.P$4
- new net AR_OUT: RN1.5, RN2.5, U$3.P$3
- new net DAC1: DAC.1, U2.20
- new net DAC2: DAC.3, U2.21
- net A4: now also U2.43
- net AB_EXT: now also RN1.2; no longer U$3.P$5
- net AG_EXT: now also RN1.3; no longer U$3.P$4
- net AR_EXT: now also RN1.4; no longer U$3.P$3
- net GND: now also DAC.2, PWR.C; no longer LED1.C
- net N$12: now also PWR.A; no longer LED1.A
- net VGND: now also RN2.1, RN2.2, RN2.3, RN2.4
- net _ACTIVE: now also U2.22
Routing:
- net _ACTIVE: track 27.5 -> 96.0 mm
- net A4: track 30.5 -> 48.2 mm, vias 1 -> 3
- net DAC2: track 0.00 -> 17.5 mm
- net N$12: track 2.63 -> 15.0 mm, vias 1 -> 0
- net AB_OUT: track 0.00 -> 12.0 mm, vias 0 -> 1
- net DAC1: track 0.00 -> 10.3 mm
- net AG_OUT: track 0.00 -> 6.59 mm
- net AR_OUT: track 0.00 -> 6.07 mm
- net _KB_CLOCK: track 112.0 -> 117.1 mm
- net VGND: track 73.8 -> 78.9 mm
- net _KB_DATA: track 83.3 -> 87.8 mm
- net AG_EXT: track 40.3 -> 36.0 mm
- net LED: track 12.4 -> 8.28 mm
- net AR_EXT: track 45.0 -> 40.9 mm
- net _TXD: track 88.6 -> 92.6 mm
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
Commit message: Resistor value cleanup
Parts:
- C13: value 10u -> 10uF
- C16: value 100n -> 100nF
- C17, C18, C19, C20, C21: value (none) -> 0.1uF
- R1: value (none) -> 4K7
- R2: value 100k -> 100K
Routing:
- net NRST: track 101.3 -> 99.7 mm

Commit message: fix vcap
Parts:
- removed RN1, RN2: (no value), resistor-dil:CAY16
- added C22: 100n, rcl:C0805
- added R10, R11, R12: 29R9, rcl:R0603
- added R6, R7, R9: 49R9, rcl:R0603
- F1, F2: value 1206L050YR -> 0R; device 1206L050YR:FUSC3216X75N -> eagle-ltspice:R1206
- LED2, PWR: value (none) -> LED
- moved R2 12.1 mm to (107.9, 54.1), turned to 180 degrees
- moved F2 1.04 mm to (18.5, 53.0)
- moved F1 0.98 mm to (18.5, 50.4)
- moved U$3 0.48 mm to (117.7, 44.4)
- renumbered XC9572XL to IC2, Y1 to X1
Connections:
- removed net VCAP_1: U2.30
- new net VCAP: C22.1, U2.30
- net AB_EXT: now also R10.1; no longer RN1.2
- net AB_OUT: now also R10.2, R9.1; no longer RN1.7, RN2.7
- net AG_EXT: now also R11.1; no longer RN1.3
- net AG_OUT: now also R11.2, R7.1; no longer RN1.6, RN2.6
- net AR_EXT: now also R12.1; no longer RN1.4
- net AR_OUT: now also R12.2, R6.1; no longer RN1.5, RN2.5
- net GND: now also C22.2, R6.2, R7.2, R9.2
- net VGND: no longer RN2.1, RN2.2, RN2.3, RN2.4
Routing:
- net NRST: track 99.7 -> 108.9 mm
- net VGND: track 78.9 -> 73.8 mm
- net VCAP: track 0.00 -> 4.12 mm, vias 0 -> 1
- net VCC33: track 114.4 -> 110.6 mm
- net GND: track 63.4 -> 66.9 mm, vias 23 -> 27
- net VCC: track 32.2 -> 35.2 mm, vias 6 -> 5
- net AB_EXT: track 44.3 -> 47.1 mm
- net +12V: track 100.3 -> 102.0 mm
- net AB_OUT: track 12.0 -> 10.6 mm, vias 1 -> 0
- net AG_OUT: track 6.59 -> 5.29 mm
- net N$1: track 6.57 -> 7.81 mm
- net N$2: track 3.37 -> 4.35 mm
- net AR_OUT: track 6.07 -> 6.98 mm
- net AR_EXT: track 40.9 -> 41.8 mm

Commit message: Added LSE oscillator. Removed TXD/RXD and added A5.
Parts:
- added C23, C24: 22p, eagle-ltspice:C0603
- added JP3: (no value), SparkFun-Retired:1X02
- added X2: SMD-CRYSTAL-32768KHZ-20PF-20PPM(2P-5.0X3.2MM), SMD-CRYSTAL-8MHZ-20PF-20PPM_2P-5.0X3.2MM_:X2-SMD-5.0X3.2X1.3MM
- C6: device eagle-ltspice:C0603 -> rcl:C0603
- moved R5 6.17 mm to (58.6, 44.4)
- moved C7 3.94 mm to (48.5, 55.7), turned to 45 degrees
- moved C10 0.82 mm to (48.4, 44.9), turned to 90 degrees
- moved C6 0.37 mm to (39.1, 51.4)
- moved C11 0.32 mm to (48.4, 48.4), turned to 270 degrees
- moved C8 0.05 mm to (39.1, 53.5)
Connections:
- removed net N$5: D1.1, G1.+, R5.2
- new net LSE_OSCIN: C23.1, U2.3, X2.2
- new net LSE_OSCOUT: C24.1, U2.4, X2.1
- new net VBAT: D1.1, G1.+, R5.2, U2.1
- net A5: now also U2.11
- net GND: now also C23.2, C24.2
- net INTSIG8: now also U2.14; no longer U2.2
- net R_W: now also U2.2; no longer U2.3
- net VCC33: no longer U2.1
- net _DSACK_0: no longer U2.4
- net _KB_DATA: now also U2.15; no longer U2.11
- net _RXD: now also JP3.2; no longer U2.14
- net _TXD: now also JP3.1; no longer U2.15
Routing:
- net VBAT: track 0.00 -> 42.2 mm, vias 0 -> 2
- net _DSACK_0: track 104.4 -> 69.3 mm
- net A5: track 35.0 -> 60.0 mm, vias 0 -> 1
- net _RXD: track 102.6 -> 81.0 mm
- net N$5: track 20.1 -> 0.00 mm
- net LSE_OSCOUT: track 0.00 -> 19.3 mm
- net _TXD: track 92.4 -> 73.5 mm
- net LSE_OSCIN: track 0.00 -> 13.0 mm
- net OSCIN: track 13.8 -> 24.4 mm
- net NRST: track 108.9 -> 112.3 mm
- net VCC33: track 110.6 -> 107.3 mm
- net R_W: track 109.1 -> 111.8 mm
- net INTSIG8: track 40.5 -> 38.1 mm, vias 0 -> 2
- net SPI2_MISO: track 40.9 -> 38.7 mm
- net GND: track 66.9 -> 68.3 mm, vias 27 -> 29
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