File: eagle/cd32_riser.brd (EAGLE design)
At the start: 124.5 x 60 mm, 57 parts, among them CN1 CD32-EXPANSION, CN2 CD32-EXPANSION, IC1 LM1117MPX-3.3, IC2 XC9572XL-VQ64, U2 STM32F722RET6, X1 SMD-CRYSTAL-8MHZ-20PF-20PPM(2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, X2 SMD-CRYSTAL-32768KHZ-20PF-20P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

Commit message: minor board changes
Parts:
- removed R10, R11, R12: 29R9, rcl:R0603
- removed R9: 49R9, rcl:R0603
- added IC4: THS7314D, THS7314D:SOIC127P599X175-8N
- R5: value 10k -> 100K
- R6, R7: value 49R9 -> 100K; device rcl:R0603 -> rcl:M0805
- moved R5 61.7 mm to (119.9, 37.9), flipped to the bottom, turned to 0 degrees
- moved R7 10.4 mm to (119.9, 42.0), flipped to the bottom, turned to 180 degrees
- moved R6 3.10 mm to (119.9, 39.9), flipped to the bottom, turned to 180 degrees
- moved U$3 2.40 mm to (116.8, 46.6)
- moved D1 1.59 mm to (55.0, 43.5), turned to 90 degrees
- renumbered U2 to IC3
Connections:
- new net N$5: D1.1, G1.+
- net AB_EXT: now also IC4.1, R5.2; no longer R10.1
- net AB_OUT: now also IC4.8; no longer R10.2, R9.1
- net AG_EXT: now also IC4.2, R6.1; no longer R11.1
- net AG_OUT: now also IC4.7; no longer R11.2, R7.1
- net AR_EXT: now also IC4.3, R7.1; no longer R12.1
- net AR_OUT: now also IC4.6; no longer R12.2, R6.1
- net GND: now also IC4.5, R5.1; no longer R9.2
- net VBAT: now also D1.3; no longer D1.1, G1.+, R5.2
- net VCC: now also IC4.4
- net VCC33: no longer D1.3, R5.1
Routing:
- net VBAT: track 42.2 -> 19.1 mm
- net +12V: track 102.0 -> 85.7 mm
- net AR_EXT: track 41.8 -> 58.0 mm, vias 0 -> 1
- net AG_EXT: track 36.2 -> 51.2 mm, vias 0 -> 1
- net AG_OUT: track 5.29 -> 18.0 mm
- net N$5: track 0.00 -> 9.79 mm
- net AB_EXT: track 47.1 -> 56.4 mm
- net AB_OUT: track 10.6 -> 18.1 mm
- net AR_OUT: track 6.98 -> 13.5 mm
- net _VSYNC: track 53.3 -> 58.9 mm
- net _HSYNC: track 56.9 -> 61.7 mm
- net NRST: track 112.3 -> 115.3 mm
- net VCC33: track 107.3 -> 104.4 mm, vias 23 -> 21
- net _CSYNC: track 49.4 -> 52.1 mm
- net GND: track 68.3 -> 70.4 mm, vias 29 -> 28
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Other:
- board text added: "3.3V"
- board text added: "RXD"
- board text added: "TCK"
- board text added: "TDI"
- board text added: "TDO"
- board text added: "TMS"
- board text added: "TXD"
- board text added: "Terrible Fire USB CD32 Adaptor (C) 2020 S.J Leary Revision 2 Published Under the GNU GPLv2"
- board text removed: "Terrible Fire USB CD32 Adaptor (C) 2020 S.J Leary Revision 1 Published Under the GNU GPLv2"

Commit message: rationalized cap sizes
Parts:
- added C25: 100n, rcl:C0603
- C1: value 100n -> 100nF; device rcl:C0805 -> rcl:C1206
- C12: device rcl:C0805 -> rcl:C0603
- C13: device rcl:C0805 -> rcl:C1206
- C15: device rcl:C0805 -> rcl:R0603
- R3, R4: device rcl:M0805 -> rcl:R0603
Connections:
- net GND: now also C25.2
- net VCC: now also C25.1
Routing:
- net VCC: track 36.8 -> 39.7 mm
- net AB_EXT: track 56.4 -> 55.3 mm
- net GND: track 70.4 -> 71.1 mm, vias 28 -> 29

Commit message: updated footprint of 32Khz crystal
Parts:
- X1: value SMD-CRYSTAL-8MHZ-20PF-20PPM(2P-5.0X3.2MM) -> SMD-CRYSTAL-25MHZ-20PF-20PPM(2P-5.0X3.2MM)
- X2: value SMD-CRYSTAL-32768KHZ-20PF-20PPM(2P-5.0X3.2MM) -> 32.768KHZ; device SMD-CRYSTAL-8MHZ-20PF-20PPM_2P-5.0X3.2MM_:X2-SMD-5.0X3.2X1.3MM -> adafruit:XTAL3215
- moved X2 0.33 mm to (48.1, 40.2), turned to 0 degrees
Connections:
- net LSE_OSCIN: now also X2.P$2; no longer X2.2
- net LSE_OSCOUT: now also X2.P$1; no longer X2.1
