File: eagle/cd32_riser.sch (EAGLE design)
At the start: 37 parts, among them CN1 CD32-EXPANSION, CN2 CD32-EXPANSION, IC1 LM1117MPX-3.3, U1 STM32F10XRXT6, X1 PN87520-S

Commit message: Added punt pullup
Parts:
- added R1: (no value), rcl:R-EU_M1206
- renumbered XC9572XL(BUS) to XC9572XL
Connections:
- net GND: now also BT1.-
- net PUNT_IN: now also R1.1
- net VCC: now also R1.2
Other:
- moved on the sheet: BT1

Commit message: Added missing 10k resistor
Parts:
- added R4: 10k, rcl:R-EU_M0805
Connections:
- new net N$4: LED2.A, R4.2
- net VCC: now also R4.1
Changed lines of the file:
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@@
 <part name="BT1" library="SparkFun-Batteries" deviceset="BATTERY" device="-20MM_PTH"/>
 <part name="R1" library="rcl" library_urn="urn:adsk.eagle:library:334" deviceset="R-EU_" device="M1206" package3d_urn="urn:adsk.eagle:package:23566/1"/>
+<part name="R4" library="rcl" library_urn="urn:adsk.eagle:library:334" deviceset="R-EU_" device="M0805" package3d_urn="urn:adsk.eagle:package:23556/1" value="10k"/>
+<part name="SUPPLY10" library="supply2" library_urn="urn:adsk.eagle:library:372" deviceset="VCC" device=""/>
 </parts>
 <sheets>
@@
 </instance>
 <instance part="BT1" gate="G$1" x="210.82" y="172.72" rot="R90"/>
+<instance part="R4" gate="G$1" x="208.28" y="93.98" rot="R180">
+<attribute name="NAME" x="212.09" y="92.4814" size="1.778" layer="95" rot="R180"/>
+<attribute name="VALUE" x="212.09" y="97.282" size="1.778" layer="96" rot="R180"/>
+</instance>
+<instance part="SUPPLY10" gate="G$1" x="220.98" y="93.98" rot="R270">
+<attribute name="VALUE" x="224.155" y="95.885" size="1.778" layer="96" rot="R270"/>
+</instance>
 </instances>
 <busses>
@@
 <pinref part="SUPPLY9" gate="G$1" pin="VCC"/>
 </segment>
+<segment>
+<pinref part="R4" gate="G$1" pin="1"/>
+<wire x1="218.44" y1="93.98" x2="213.36" y2="93.98" width="0.1524" layer="91"/>
+<pinref part="SUPPLY10" gate="G$1" pin="VCC"/>
+</segment>
 </net>
 <net name="SWDIO" class="0">
@@
 </segment>
 </net>
+<net name="N$4" class="0">
+<segment>
+<pinref part="R4" gate="G$1" pin="2"/>
+<pinref part="LED2" gate="G$1" pin="A"/>
+<wire x1="203.2" y1="93.98" x2="195.58" y2="93.98" width="0.1524" layer="91"/>
+</segment>
+</net>

Commit message: Added missing 10k resistor
Parts:
- added D1: BAT54, diode:BAT54
- added R5: 10k, rcl:R-EU_M0805
Connections:
- new net N$5: BT1.+, D1.A, R5.2
- net VCC33: now also D1.C, R5.1
Changed lines of the file:
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@@
 <part name="R4" library="rcl" library_urn="urn:adsk.eagle:library:334" deviceset="R-EU_" device="M0805" package3d_urn="urn:adsk.eagle:package:23556/1" value="10k"/>
 <part name="SUPPLY10" library="supply2" library_urn="urn:adsk.eagle:library:372" deviceset="VCC" device=""/>
+<part name="R5" library="rcl" library_urn="urn:adsk.eagle:library:334" deviceset="R-EU_" device="M0805" package3d_urn="urn:adsk.eagle:package:23556/1" value="10k"/>
+<part name="D1" library="diode" library_urn="urn:adsk.eagle:library:210" deviceset="BAT54" device="" package3d_urn="urn:adsk.eagle:package:43389/2"/>
 </parts>
 <sheets>
@@
 <attribute name="VALUE" x="224.155" y="95.885" size="1.778" layer="96" rot="R270"/>
 </instance>
+<instance part="R5" gate="G$1" x="187.96" y="180.34" rot="R270">
+<attribute name="NAME" x="189.4586" y="184.15" size="1.778" layer="95" rot="R270"/>
+<attribute name="VALUE" x="184.658" y="184.15" size="1.778" layer="96" rot="R270"/>
+</instance>
+<instance part="D1" gate="G$1" x="182.88" y="167.64" rot="R180"/>
 </instances>
 <busses>
@@
 <junction x="27.94" y="185.42"/>
 <wire x1="27.94" y1="185.42" x2="20.32" y2="185.42" width="0.1524" layer="91"/>
+<pinref part="R5" gate="G$1" pin="1"/>
+<wire x1="160.02" y1="185.42" x2="175.26" y2="185.42" width="0.1524" layer="91"/>
+<junction x="160.02" y="185.42"/>
+<pinref part="D1" gate="G$1" pin="C"/>
+<wire x1="175.26" y1="185.42" x2="187.96" y2="185.42" width="0.1524" layer="91"/>
+<wire x1="180.34" y1="167.64" x2="175.26" y2="167.64" width="0.1524" layer="91"/>
+<wire x1="175.26" y1="167.64" x2="175.26" y2="185.42" width="0.1524" layer="91"/>
+<junction x="175.26" y="185.42"/>
 </segment>
 <segment>
@@
 <segment>
 <pinref part="U1" gate="PORTA_H" pin="PA11"/>
-<wire x1="157.48" y1="27.94" x2="149.86" y2="27.94" width="0.1524" layer="91"/>
-<label x="142.24" y="27.94" size="1.778" layer="95"/>
+<wire x1="157.48" y1="27.94" x2="137.16" y2="27.94" width="0.1524" layer="91"/>
+<label x="137.16" y="27.94" size="1.778" layer="95"/>
 </segment>
 <segment>
@@
 <segment>
 <pinref part="U1" gate="PORTA_H" pin="PA12"/>
-<wire x1="157.48" y1="25.4" x2="149.86" y2="25.4" width="0.1524" layer="91"/>
-<label x="142.24" y="25.4" size="1.778" layer="95"/>
+<wire x1="157.48" y1="25.4" x2="137.16" y2="25.4" width="0.1524" layer="91"/>
+<label x="137.16" y="25.4" size="1.778" layer="95"/>
 </segment>
 <segment>
@@
 </segment>
 </net>
+<net name="N$5" class="0">
+<segment>
+<pinref part="R5" gate="G$1" pin="2"/>
+<pinref part="D1" gate="G$1" pin="A"/>
+<wire x1="187.96" y1="175.26" x2="187.96" y2="167.64" width="0.1524" layer="91"/>
+<wire x1="187.96" y1="167.64" x2="185.42" y2="167.64" width="0.1524" layer="91"/>
+<pinref part="BT1" gate="G$1" pin="+"/>
+<wire x1="187.96" y1="167.64" x2="210.82" y2="167.64" width="0.1524" layer="91"/>
+<junction x="187.96" y="167.64"/>
+</segment>
+</net>

Commit message: decoupling for the CPLD.
Parts:
- added C17, C18, C19, C20, C21: (no value), rcl:C-EUC0603
Connections:
- net GND: now also C17.2, C18.2, C19.2, C20.2, C21.2
- net VCC33: now also C17.1, C18.1, C19.1, C20.1, C21.1
Changed lines of the file:
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@@
 <part name="R5" library="rcl" library_urn="urn:adsk.eagle:library:334" deviceset="R-EU_" device="M0805" package3d_urn="urn:adsk.eagle:package:23556/1" value="10k"/>
 <part name="D1" library="diode" library_urn="urn:adsk.eagle:library:210" deviceset="BAT54" device="" package3d_urn="urn:adsk.eagle:package:43389/2"/>
+<part name="C17" library="rcl" library_urn="urn:adsk.eagle:library:334" deviceset="C-EU" device="C0603" package3d_urn="urn:adsk.eagle:package:23616/2"/>
+<part name="C18" library="rcl" library_urn="urn:adsk.eagle:library:334" deviceset="C-EU" device="C0603" package3d_urn="urn:adsk.eagle:package:23616/2"/>
+<part name="C19" library="rcl" library_urn="urn:adsk.eagle:library:334" deviceset="C-EU" device="C0603" package3d_urn="urn:adsk.eagle:package:23616/2"/>
+<part name="C20" library="rcl" library_urn="urn:adsk.eagle:library:334" deviceset="C-EU" device="C0603" package3d_urn="urn:adsk.eagle:package:23616/2"/>
+<part name="C21" library="rcl" library_urn="urn:adsk.eagle:library:334" deviceset="C-EU" device="C0603" package3d_urn="urn:adsk.eagle:package:23616/2"/>
 </parts>
 <sheets>
@@
 <instance part="XC9572XL" gate="XC9572XL-VQ64" x="106.68" y="86.36" rot="R180"/>
 <instance part="R1" gate="G$1" x="43.18" y="157.48" rot="R90"/>
+<instance part="C17" gate="G$1" x="142.24" y="170.18"/>
+<instance part="C18" gate="G$1" x="152.4" y="170.18"/>
+<instance part="C19" gate="G$1" x="162.56" y="170.18"/>
+<instance part="C20" gate="G$1" x="172.72" y="170.18"/>
+<instance part="C21" gate="G$1" x="182.88" y="170.18"/>
 </instances>
 <busses>
@@
 <label x="33.02" y="96.52" size="1.778" layer="95"/>
 </segment>
+<segment>
+<pinref part="C17" gate="G$1" pin="2"/>
+<wire x1="195.58" y1="157.48" x2="182.88" y2="157.48" width="0.1524" layer="91"/>
+<wire x1="182.88" y1="157.48" x2="172.72" y2="157.48" width="0.1524" layer="91"/>
+<wire x1="172.72" y1="157.48" x2="162.56" y2="157.48" width="0.1524" layer="91"/>
+<wire x1="162.56" y1="157.48" x2="152.4" y2="157.48" width="0.1524" layer="91"/>
+<wire x1="152.4" y1="157.48" x2="142.24" y2="157.48" width="0.1524" layer="91"/>
+<wire x1="142.24" y1="157.48" x2="142.24" y2="165.1" width="0.1524" layer="91"/>
+<pinref part="C18" gate="G$1" pin="2"/>
+<wire x1="152.4" y1="165.1" x2="152.4" y2="157.48" width="0.1524" layer="91"/>
+<junction x="152.4" y="157.48"/>
+<pinref part="C19" gate="G$1" pin="2"/>
+<wire x1="162.56" y1="165.1" x2="162.56" y2="157.48" width="0.1524" layer="91"/>
+<junction x="162.56" y="157.48"/>
+<pinref part="C20" gate="G$1" pin="2"/>
+<wire x1="172.72" y1="165.1" x2="172.72" y2="157.48" width="0.1524" layer="91"/>
+<junction x="172.72" y="157.48"/>
+<pinref part="C21" gate="G$1" pin="2"/>
+<wire x1="182.88" y1="165.1" x2="182.88" y2="157.48" width="0.1524" layer="91"/>
+<junction x="182.88" y="157.48"/>
+</segment>
 </net>
 <net name="VCC33" class="0">
@@
 <label x="165.1" y="83.82" size="1.778" layer="95"/>
 </segment>
+<segment>
+<pinref part="C17" gate="G$1" pin="1"/>
+<wire x1="142.24" y1="180.34" x2="142.24" y2="172.72" width="0.1524" layer="91"/>
+</segment>
+<segment>
+<pinref part="C18" gate="G$1" pin="1"/>
+<wire x1="152.4" y1="180.34" x2="152.4" y2="172.72" width="0.1524" layer="91"/>
+</segment>
+<segment>
+<wire x1="162.56" y1="180.34" x2="162.56" y2="172.72" width="0.1524" layer="91"/>
+<pinref part="C19" gate="G$1" pin="1"/>
+</segment>
+<segment>
+<wire x1="172.72" y1="180.34" x2="172.72" y2="172.72" width="0.1524" layer="91"/>
+<pinref part="C20" gate="G$1" pin="1"/>
+</segment>
+<segment>
+<wire x1="182.88" y1="180.34" x2="182.88" y2="172.72" width="0.1524" layer="91"/>
+<pinref part="C21" gate="G$1" pin="1"/>
+</segment>
 </net>

Commit message: updated the arm side of stuff significantly
Parts:
- removed BT1: (no value), SparkFun-Batteries:BATTERY-20MM_PTH
- removed Q1: (no value), crystal:CRYSTALHC49S
- removed SJ1, SJ2, SJ3, SJ4: (no value), jumper:SJ2W
- removed U1: STM32F10XRXT6, stm32:STM32F10XRXT6
- removed X1: PN87520-S, con-berg:PN87520-S
- added G1: CH23-1220LF, battery:CH23-1220LF
- added JP1: (no value), SparkFun-Retired:JUMPER-2PTH
- added U$1: USB-A-2_USB_USB-A-2, board:USB-A-2_USB_USB-A-2
- added U2: STM32F722RET6, STM32F722RET6:STM32F722RET6
- added Y1: SMD-CRYSTAL-8MHZ-20PF-20PPM(2P-5.0X3.2MM), SMD-CRYSTAL-8MHZ-20PF-20PPM_2P-5.0X3.2MM_:SMD-CRYSTAL-8MHZ-20PF-20PPM(2P-5.0X3.2MM)
Connections:
- removed net N$1: C10.1, Q1.2, U1PORTD/OSC.PD0/OSC<=
- removed net N$10: SJ3.2, U1PORTC_L.PC7
- removed net N$11: SJ2.2, U1PORTC_H.PC8
- removed net N$2: C11.1, Q1.1, U1PORTD/OSC.PD1/OSC=>
- removed net N$3: BOOT0.2, U1RESET.BOOT0
- removed net N$6: SJ1.2, U1PORTC_H.PC9
- removed net N$8: LED2.C, U1PORTB_H.PB10
- removed net N$9: SJ4.2, U1PORTC_L.PC6
- removed net SPI_NSS: U1PORTA_H.PA15, XC9572XL.PB03/5
- removed net USB_DM: U1PORTA_H.PA11, X1.2
- removed net USB_DP: U1PORTA_H.PA12, X1.3
- new net BOOT: BOOT0.2, U2.BOOT
- new net INTSIG0: U2.PB8, XC9572XL.PB03/2
- new net INTSIG1: U2.PB9, XC9572XL.PB01/17
- new net INTSIG2: U2.PB12, XC9572XL.PB01/12
- new net INTSIG3: U2.PA15(JTDI), XC9572XL.PB03/5
- new net INTSIG4: U2.PC8, XC9572XL.PB01/4
- new net INTSIG5: U2.PC9, XC9572XL.PB01/3
- new net INTSIG6: U2.PC10, XC9572XL.PB01/8
- new net INTSIG7: U2.PC11, XC9572XL.PB01/6
- new net INTSIG8: U2.PC13, XC9572XL.PB01/14
- new net LED: LED2.C, U2.PB11
- new net OSCIN: C10.1, U2.PH0-OSC_IN, Y1.2
- new net OSCOUT: C11.1, U2.PH1-OSC_OUT, Y1.1
- new net USB1_DM: U$1-B.2-2, U2.PA11
- new net USB1_DP: U$1-B.2-3, U2.PA12
- new net USB2_DM: U$1-A.1-2, U2.PB14
- new net USB2_DP: U$1-A.1-3, U2.PB15
- net AB: no longer U$3.P$5
- net AB_EXT: now also U$3.P$5
- net AG: no longer U$3.P$4
- net AG_EXT: now also U$3.P$4
- net AR: no longer U$3.P$3
- net AR_EXT: now also U$3.P$3
- net D24: now also U2.PB0
- net D25: now also U2.PB1
- net D26: now also U2.PB2
- net D27: now also U2.PB3(JTDO/TRACESWO)
- net D28: now also U2.PB4(!JTRST)
- net D29: now also U2.PB5
- net D30: now also U2.PB6
- net D31: now also U2.PB7
- net DKWE: now also U2.PA6
- net GND: now also G1.-, U$1-A.1-4, U$1-B.2-4, U$1SHIELD.SHIELD1, U$1SHIELD.SHIELD2, U$1SHIELD.SHIELD3, U$1SHIELD.SHIELD4, U2.VSS, U2.VSSA; no longer BT1.-, SJ1.1, SJ2.1, SJ3.1, SJ4.1, U1AN_POWER.VSSA, U1PORTA_L.PA2, U1PORTB_L.PB2, U1POWER.VSS_1, U1POWER.VSS_2, U1POWER.VSS_3, U1POWER.VSS_4, X1.4
- net N$5: now also G1.+; no longer BT1.+
- net NRST: now also U2.!RST; no longer U1RESET.NRST
- net PA9BOOT: now also U2.PA9; no longer U1PORTA_H.PA9
- net PUNT_IN: now also XC9572XL.PB01/5; no longer XC9572XL.PB01/4
- net PUNT_OUT: now also XC9572XL.PB01/2; no longer XC9572XL.PB01/6
- net R_W: now also U2.PC14-OSC32_IN, XC9572XL.PB02/14; no longer XC9572XL.PB02/17
- net SIZ0: no longer XC9572XL.PB02/12
- net SIZ1: no longer XC9572XL.PB02/11
- net SPI_CK: now also U2.PC0, XC9572XL.PB01/15; no longer U1PORTB_L.PB3, XC9572XL.PB01/17
- net SPI_MISO: now also U2.PC2, XC9572XL.PB01/10; no longer U1PORTB_L.PB4, XC9572XL.PB01/15
- net SPI_MOSI: now also U2.PC3, XC9572XL.GCLK2; no longer U1PORTB_L.PB5, XC9572XL.PB01/10
- net SWCLK: now also U2.PA14(JTCK-SWCLK); no longer U1PORTA_H.PA14
- net SWDIO: now also U2.PA13(JTMS-SWDIO); no longer U1PORTA_H.PA13
- net UART5_RX: now also JP1.1, U2.PD2; no longer U1PORTD/OSC.PD2, XC9572XL.PB03/2
- net UART5_TX: now also JP1.2, U2.PC12; no longer U1PORTC_H.PC12, XC9572XL.PB01/12
- net VCC: now also U$1-A.1-1, U$1-B.2-1; no longer X1.1
- net VCC33: now also U2.VBAT, U2.VDD, U2.VREF+; no longer SJ1.3, SJ2.3, SJ3.3, SJ4.3, U1AN_POWER.VBAT, U1AN_POWER.VDDA, U1POWER.VDD_1, U1POWER.VDD_2, U1POWER.VDD_3, U1POWER.VDD_4
- net _AS: now also XC9572XL.PB02/11; no longer XC9572XL.PB02/14
- net _DKRD: now also U2.PA7
- net _DKWD: now also U2.PA8
- net _DS: now also XC9572XL.PB02/12; no longer XC9572XL.PB02/15
- net _DSACK_0: now also U2.PC15-OSC32_OUT, XC9572XL.PB02/17; no longer XC9572XL.PB01/5
- net _DSACK_1: now also XC9572XL.PB02/15; no longer XC9572XL.PB01/2
- net _FIRE0: now also U2.PA4
- net _FIRE1: now also U2.PA5
- net _KB_CLOCK: now also U2.PB10; no longer XC9572XL.PB01/8
- net _KB_DATA: now also U2.PC1; no longer XC9572XL.PB01/3
- net _RXD: now also U2.PA0-WKUP; no longer XC9572XL.GCLK2
- net _TXD: now also U2.PA1; no longer XC9572XL.PB01/14
Other:
- note added: "Debug Console"
- note added: "UART4"
- note removed: "BOOT1"
- note removed: "PA2-> L "Deluxe Board" PA2-> H "Basic Board""
- moved on the sheet: BOOT0, C1, C10, C11, C12, C13, C14, C15, C16, C2, C3, C4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

Commit message: updated the circuit and added fuses
Parts:
- added F1, F2: 1206L050YR, 1206L050YR:1206L050YR
Connections:
- net INTSIG0 renamed BUS_INT
- net SPI_MISO renamed SPI2_MISO
- removed net SPI_CK: U2.PC0, XC9572XL.PB01/15
- removed net SPI_MOSI: U2.PC3, XC9572XL.GCLK2
- new net N$1: F1.2, U$1-B.2-1
- new net N$2: F2.2, U$1-A.1-1
- new net SPI2_CK: U2.PB10, XC9572XL.PB01/15
- new net SPI2_MOSI: U2.PC1, XC9572XL.GCLK2
- net DKWE: now also U2.PA2; no longer U2.PA6
- net LED: now also U2.PB13; no longer U2.PB11
- net VCC: now also F1.1, F2.1; no longer U$1-A.1-1, U$1-B.2-1
- net _FIRE0: now also U2.PA3; no longer U2.PA4
- net _FIRE1: now also U2.PC0; no longer U2.PA5
- net _KB_CLOCK: now also U2.PB11; no longer U2.PB10
- net _KB_DATA: now also U2.PC3; no longer U2.PC1
Other:
- moved on the sheet: U$1-A, U$1-B

Commit message: added the address lines
Connections:
- net A0: now also U2.PC4
- net A1: now also U2.PC6
- net A2: now also U2.PC7
- net INTSIG8: now also XC9572XL.PB01/10; no longer XC9572XL.PB01/14
- net SPI2_CK: now also XC9572XL.GCLK2; no longer XC9572XL.PB01/15
- net SPI2_MISO: now also XC9572XL.PB01/15; no longer XC9572XL.PB01/10
- net SPI2_MOSI: now also XC9572XL.PB01/14; no longer XC9572XL.GCLK2
Changed lines of the file:
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@@
+</segment>
+</net>
+<net name="A0" class="0">
+<segment>
+<pinref part="U2" gate="G$1" pin="PC4"/>
+<wire x1="35.56" y1="116.84" x2="10.16" y2="116.84" width="0.1524" layer="91"/>
+<label x="17.78" y="116.84" size="1.778" layer="95"/>
+</segment>
+</net>
+<net name="A1" class="0">
+<segment>
+<pinref part="U2" gate="G$1" pin="PC6"/>
+<wire x1="35.56" y1="114.3" x2="10.16" y2="114.3" width="0.1524" layer="91"/>
+<label x="17.78" y="114.3" size="1.778" layer="95"/>
+</segment>
+</net>
+<net name="A2" class="0">
+<segment>
+<pinref part="U2" gate="G$1" pin="PC7"/>
+<wire x1="35.56" y1="111.76" x2="10.16" y2="111.76" width="0.1524" layer="91"/>
+<label x="17.78" y="111.76" size="1.778" layer="95"/>
 </segment>
 </net>
@@
 </segment>
 </net>
-<net name="SPI2_CK" class="0">
+<net name="SPI2_MISO" class="0">
 <segment>
 <wire x1="12.7" y1="101.6" x2="71.12" y2="101.6" width="0.1524" layer="91"/>
@@
 </segment>
 </net>
-<net name="SPI2_MISO" class="0">
-<segment>
-<wire x1="12.7" y1="104.14" x2="71.12" y2="104.14" width="0.1524" layer="91"/>
-<pinref part="XC9572XL" gate="XC9572XL-VQ64" pin="PB01/10"/>
-<label x="33.02" y="104.14" size="1.778" layer="95"/>
-</segment>
-</net>
 <net name="SPI2_MOSI" class="0">
 <segment>
-<wire x1="86.36" y1="180.34" x2="86.36" y2="121.92" width="0.1524" layer="91"/>
-<pinref part="XC9572XL" gate="XC9572XL-VQ64" pin="GCLK2"/>
-<label x="86.36" y="144.78" size="1.778" layer="95" rot="R90"/>
+<wire x1="12.7" y1="106.68" x2="71.12" y2="106.68" width="0.1524" layer="91"/>
+<pinref part="XC9572XL" gate="XC9572XL-VQ64" pin="PB01/14"/>
+<label x="33.02" y="106.68" size="1.778" layer="95"/>
 </segment>
 </net>
@@
 <net name="INTSIG8" class="0">
 <segment>
-<wire x1="71.12" y1="106.68" x2="12.7" y2="106.68" width="0.1524" layer="91"/>
-<pinref part="XC9572XL" gate="XC9572XL-VQ64" pin="PB01/14"/>
-<label x="33.02" y="106.68" size="1.778" layer="95"/>
+<wire x1="71.12" y1="104.14" x2="12.7" y2="104.14" width="0.1524" layer="91"/>
+<pinref part="XC9572XL" gate="XC9572XL-VQ64" pin="PB01/10"/>
+<label x="33.02" y="104.14" size="1.778" layer="95"/>
 </segment>
 </net>
@@
 </segment>
 </net>
+<net name="SPI2_CK" class="0">
+<segment>
+<pinref part="XC9572XL" gate="XC9572XL-VQ64" pin="GCLK2"/>
+<wire x1="86.36" y1="121.92" x2="86.36" y2="180.34" width="0.1524" layer="91"/>
+<wire x1="86.36" y1="180.34" x2="83.82" y2="180.34" width="0.1524" layer="91"/>
+<label x="86.36" y="144.78" size="1.778" layer="95" rot="R90"/>
+</segment>
+</net>

Commit message: finished the route
Parts:
- added DAC: JUMPER-3PTH, SparkFun-Retired:JUMPER-3PTH
- added RN1, RN2: (no value), resistor-dil:4R-NCAY16
- renumbered LED1 to PWR
Connections:
- new net AB_OUT: RN1B.2, RN2B.2, U$3.P$5
- new net AG_OUT: RN1C.2, RN2C.2, U$3.P$4
- new net AR_OUT: RN1D.2, RN2D.2, U$3.P$3
- new net DAC1: DAC.1, U2.PA4
- new net DAC2: DAC.3, U2.PA5
- net A4: now also U2.PA10
- net AB_EXT: now also RN1B.1; no longer U$3.P$5
- net AG_EXT: now also RN1C.1; no longer U$3.P$4
- net AR_EXT: now also RN1D.1; no longer U$3.P$3
- net GND: now also DAC.2
- net VGND: now also RN2A.1, RN2B.1, RN2C.1, RN2D.1
- net _ACTIVE: now also U2.PA6
