File: eagle/cd32_riser.sch (EAGLE design)
At the start: 48 parts, among them CN1 CD32-EXPANSION, CN2 CD32-EXPANSION, IC1 LM1117MPX-3.3, U2 STM32F722RET6, Y1 SMD-CRYSTAL-8MHZ-20PF-20PPM(2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

Commit message: Resistor value cleanup
Parts:
- C13: value 10u -> 10uF
- C16: value 100n -> 100nF
- C17, C18, C19, C20, C21: value (none) -> 0.1uF
- R1: value (none) -> 4K7
- R2: value 100k -> 100K
Changed lines of the file:
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@@
 <?xml version="1.0" encoding="utf-8"?>
 <!DOCTYPE eagle SYSTEM "eagle.dtd">
-<eagle version="8.7.1">
+<eagle version="9.6.0">
 <drawing>
 <settings>
@@
 <part name="CN1" library="Amiga" deviceset="CD32-EXPANSION" device=""/>
 <part name="CN2" library="Amiga" deviceset="CD32-EXPANSION" device=""/>
-<part name="C16" library="eagle-ltspice" library_urn="urn:adsk.eagle:library:217" deviceset="C" device="C0603" package3d_urn="urn:adsk.eagle:package:13262/1" value="100n"/>
+<part name="C16" library="eagle-ltspice" library_urn="urn:adsk.eagle:library:217" deviceset="C" device="C0603" package3d_urn="urn:adsk.eagle:package:13262/1" value="100nF"/>
 <part name="GND5" library="supply1" library_urn="urn:adsk.eagle:library:371" deviceset="GND" device=""/>
 <part name="C14" library="eagle-ltspice" library_urn="urn:adsk.eagle:library:217" deviceset="C" device="C0603" package3d_urn="urn:adsk.eagle:package:13262/1" value="100n"/>
@@
 <part name="C7" library="eagle-ltspice" library_urn="urn:adsk.eagle:library:217" deviceset="C" device="C0603" package3d_urn="urn:adsk.eagle:package:13262/1" value="100n"/>
 <part name="GND3" library="supply1" library_urn="urn:adsk.eagle:library:371" deviceset="GND" device=""/>
-<part name="R2" library="rcl" library_urn="urn:adsk.eagle:library:334" deviceset="R-EU_" device="M0805" package3d_urn="urn:adsk.eagle:package:23556/1" value="100k"/>
+<part name="R2" library="rcl" library_urn="urn:adsk.eagle:library:334" deviceset="R-EU_" device="M0805" package3d_urn="urn:adsk.eagle:package:23556/1" value="100K"/>
 <part name="SUPPLY4" library="supply2" library_urn="urn:adsk.eagle:library:372" deviceset="VDD" device=""/>
 <part name="SUPPLY5" library="supply2" library_urn="urn:adsk.eagle:library:372" deviceset="VCC" device=""/>
@@
 <part name="C3" library="eagle-ltspice" library_urn="urn:adsk.eagle:library:217" deviceset="C" device="C0603" package3d_urn="urn:adsk.eagle:package:13262/1" value="10u"/>
 <part name="C1" library="rcl" library_urn="urn:adsk.eagle:library:334" deviceset="C-EU" device="C0805" package3d_urn="urn:adsk.eagle:package:23617/2" value="100n"/>
-<part name="C13" library="rcl" library_urn="urn:adsk.eagle:library:334" deviceset="C-EU" device="C0805" package3d_urn="urn:adsk.eagle:package:23617/2" value="10u"/>
+<part name="C13" library="rcl" library_urn="urn:adsk.eagle:library:334" deviceset="C-EU" device="C0805" package3d_urn="urn:adsk.eagle:package:23617/2" value="10uF"/>
 <part name="C15" library="rcl" library_urn="urn:adsk.eagle:library:334" deviceset="C-EU" device="C0805" package3d_urn="urn:adsk.eagle:package:23617/2" value="100n"/>
 <part name="LED2" library="led" library_urn="urn:adsk.eagle:library:259" deviceset="LED" device="SML0805" package3d_urn="urn:adsk.eagle:package:15830/1"/>
@@
 <part name="JTAG" library="microbuilder" deviceset="HEADER-1X6" device="ROUND" value="JTAG"/>
 <part name="XC9572XL" library="terriblefire" deviceset="XC9572XL-VQ64" device=""/>
-<part name="R1" library="rcl" library_urn="urn:adsk.eagle:library:334" deviceset="R-EU_" device="M1206" package3d_urn="urn:adsk.eagle:package:23566/1"/>
+<part name="R1" library="rcl" library_urn="urn:adsk.eagle:library:334" deviceset="R-EU_" device="M1206" package3d_urn="urn:adsk.eagle:package:23566/1" value="4K7"/>
 <part name="R4" library="rcl" library_urn="urn:adsk.eagle:library:334" deviceset="R-EU_" device="M0805" package3d_urn="urn:adsk.eagle:package:23556/1" value="10k"/>
 <part name="SUPPLY10" library="supply2" library_urn="urn:adsk.eagle:library:372" deviceset="VCC" device=""/>
 <part name="R5" library="rcl" library_urn="urn:adsk.eagle:library:334" deviceset="R-EU_" device="M0805" package3d_urn="urn:adsk.eagle:package:23556/1" value="10k"/>
 <part name="D1" library="diode" library_urn="urn:adsk.eagle:library:210" deviceset="BAT54" device="" package3d_urn="urn:adsk.eagle:package:43389/2"/>
-<part name="C17" library="rcl" library_urn="urn:adsk.eagle:library:334" deviceset="C-EU" device="C0603" package3d_urn="urn:adsk.eagle:package:23616/2"/>
-<part name="C18" library="rcl" library_urn="urn:adsk.eagle:library:334" deviceset="C-EU" device="C0603" package3d_urn="urn:adsk.eagle:package:23616/2"/>
-<part name="C19" library="rcl" library_urn="urn:adsk.eagle:library:334" deviceset="C-EU" device="C0603" package3d_urn="urn:adsk.eagle:package:23616/2"/>
-<part name="C20" library="rcl" library_urn="urn:adsk.eagle:library:334" deviceset="C-EU" device="C0603" package3d_urn="urn:adsk.eagle:package:23616/2"/>
-<part name="C21" library="rcl" library_urn="urn:adsk.eagle:library:334" deviceset="C-EU" device="C0603" package3d_urn="urn:adsk.eagle:package:23616/2"/>
+<part name="C17" library="rcl" library_urn="urn:adsk.eagle:library:334" deviceset="C-EU" device="C0603" package3d_urn="urn:adsk.eagle:package:23616/2" value="0.1uF"/>
+<part name="C18" library="rcl" library_urn="urn:adsk.eagle:library:334" deviceset="C-EU" device="C0603" package3d_urn="urn:adsk.eagle:package:23616/2" value="0.1uF"/>
+<part name="C19" library="rcl" library_urn="urn:adsk.eagle:library:334" deviceset="C-EU" device="C0603" package3d_urn="urn:adsk.eagle:package:23616/2" value="0.1uF"/>
+<part name="C20" library="rcl" library_urn="urn:adsk.eagle:library:334" deviceset="C-EU" device="C0603" package3d_urn="urn:adsk.eagle:package:23616/2" value="0.1uF"/>
+<part name="C21" library="rcl" library_urn="urn:adsk.eagle:library:334" deviceset="C-EU" device="C0603" package3d_urn="urn:adsk.eagle:package:23616/2" value="0.1uF"/>
 <part name="U2" library="STM32F722RET6" deviceset="STM32F722RET6" device=""/>
 <part name="G1" library="battery" library_urn="urn:adsk.eagle:library:109" deviceset="CH23-1220LF" device="" package3d_urn="urn:adsk.eagle:package:4614/1"/>
@@
 <attribute name="NAME" x="317.5" y="103.632" size="1.778" layer="95"/>
 </instance>
-<instance part="RN2" gate="A" x="309.88" y="129.54" rot="R180"/>
-<instance part="RN2" gate="B" x="309.88" y="134.62" rot="R180"/>
+<instance part="RN2" gate="A" x="309.88" y="129.54" smashed="yes" rot="R180">
+<attribute name="VALUE" x="307.34" y="132.588" size="1.778" layer="96" rot="R180"/>
+<attribute name="NAME" x="314.96" y="132.588" size="1.778" layer="95" rot="R180"/>
+</instance>
+<instance part="RN2" gate="B" x="309.88" y="134.62" smashed="yes" rot="R180">
+<attribute name="VALUE" x="307.34" y="137.668" size="1.778" layer="96" rot="R180"/>
+<attribute name="NAME" x="314.96" y="137.668" size="1.778" layer="95" rot="R180"/>
+</instance>
 <instance part="RN2" gate="C" x="309.88" y="139.7" smashed="yes" rot="R180">
 <attribute name="VALUE" x="307.34" y="142.748" size="1.778" layer="96" rot="R180"/>
 <attribute name="NAME" x="314.96" y="142.748" size="1.778" layer="95" rot="R180"/>
 </instance>
-<instance part="RN2" gate="D" x="309.88" y="144.78" rot="R180"/>
+<instance part="RN2" gate="D" x="309.88" y="144.78" smashed="yes" rot="R180">
+<attribute name="VALUE" x="307.34" y="147.828" size="1.778" layer="96" rot="R180"/>
+<attribute name="NAME" x="314.96" y="147.828" size="1.778" layer="95" rot="R180"/>
+</instance>
 </instances>
 <busses>
@@
 <attribute name="VALUE" x="120.65" y="88.9" size="1.778" layer="96" align="center-left"/>
 </instance>
-<instance part="DAC" gate="G$1" x="160.02" y="175.26" rot="R270"/>
+<instance part="DAC" gate="G$1" x="160.02" y="175.26" smashed="yes" rot="R270">
+<attribute name="NAME" x="160.02" y="176.53" size="1.778" layer="95"/>
+<attribute name="VALUE" x="160.02" y="167.005" size="1.778" layer="96"/>
+</instance>
 </instances>
 <busses>

Commit message: fix vcap
Parts:
- removed RN1, RN2: (no value), resistor-dil:4R-NCAY16
- added C22: 100n, rcl:C-EUC0805
- added R10, R11, R12: 29R9, rcl:R-EU_R0603
- added R6, R7, R9: 49R9, rcl:R-EU_R0603
- F1, F2: value 1206L050YR -> 0R; device 1206L050YR:1206L050YR -> eagle-ltspice:RR1206
- LED2, PWR: value (none) -> LED
- renumbered XC9572XL to IC2, Y1 to X1
Connections:
- new net VCAP: C22.1, U2.VCAP_1
- net AB_EXT: now also R10.1; no longer RN1B.1
- net AB_OUT: now also R10.2, R9.1; no longer RN1B.2, RN2B.2
- net AG_EXT: now also R11.1; no longer RN1C.1
- net AG_OUT: now also R11.2, R7.1; no longer RN1C.2, RN2C.2
- net AR_EXT: now also R12.1; no longer RN1D.1
- net AR_OUT: now also R12.2, R6.1; no longer RN1D.2, RN2D.2
- net GND: now also C22.2, R6.2, R7.2, R9.2
- net VGND: no longer RN2A.1, RN2B.1, RN2C.1, RN2D.1

Commit message: Added LSE oscillator. Removed TXD/RXD and added A5.
Parts:
- added C23, C24: 22p, eagle-ltspice:CC0603
- added JP3: (no value), SparkFun-Retired:JUMPER-2PTH
- added X2: SMD-CRYSTAL-32768KHZ-20PF-20PPM(2P-5.0X3.2MM), SMD-CRYSTAL-8MHZ-20PF-20PPM_2P-5.0X3.2MM_:SMD-CRYSTAL-8MHZ-20PF-20PPM(2P-5.0X3.2MM)
- C6: device eagle-ltspice:CC0603 -> rcl:C-EUC0603
Connections:
- removed net N$5: D1.A, G1.+, R5.2
- new net LSE_OSCIN: C23.1, U2.PC14-OSC32_IN, X2.2
- new net LSE_OSCOUT: C24.1, U2.PC15-OSC32_OUT, X2.1
- new net VBAT: D1.A, G1.+, R5.2, U2.VBAT
- net A5: now also U2.PC3
- net GND: now also C23.2, C24.2
- net INTSIG8: now also U2.PA0-WKUP; no longer U2.PC13
- net R_W: now also U2.PC13; no longer U2.PC14-OSC32_IN
- net VCC33: no longer U2.VBAT
- net _DSACK_0: no longer U2.PC15-OSC32_OUT
- net _KB_DATA: now also U2.PA1; no longer U2.PC3
- net _RXD: now also JP3.2; no longer U2.PA0-WKUP
- net _TXD: now also JP3.1; no longer U2.PA1
Other:
- note removed: "UART4"

Commit message: minor board changes
Parts:
- removed R10, R11, R12: 29R9, rcl:R-EU_R0603
- removed R9: 49R9, rcl:R-EU_R0603
- added IC4: THS7314D, THS7314D:THS7314D
- R5: value 10k -> 100K
- R6, R7: value 49R9 -> 100K; device rcl:R-EU_R0603 -> rcl:R-EU_M0805
- renumbered U2 to IC3
Connections:
- new net N$5: D1.A, G1.+
- net AB_EXT: now also IC4.CH_1_IN, R5.2; no longer R10.1
- net AB_OUT: now also IC4.CH_1_OUT; no longer R10.2, R9.1
- net AG_EXT: now also IC4.CH_2_IN, R6.1; no longer R11.1
- net AG_OUT: now also IC4.CH_2_OUT; no longer R11.2, R7.1
- net AR_EXT: now also IC4.CH_3_IN, R7.1; no longer R12.1
- net AR_OUT: now also IC4.CH_3_OUT; no longer R12.2, R6.1
- net GND: now also IC4.GND, R5.1; no longer R9.2
- net VBAT: now also D1.C; no longer D1.A, G1.+, R5.2
- net VCC: now also IC4.VS_P
- net VCC33: no longer D1.C, R5.1
Other:
- moved on the sheet: R5

Commit message: rationalized cap sizes
Parts:
- added C25: 100n, rcl:C-EUC0603
- C1: value 100n -> 100nF; device rcl:C-EUC0805 -> rcl:C-EUC1206
- C12: device rcl:C-EUC0805 -> rcl:C-EUC0603
- C13: device rcl:C-EUC0805 -> rcl:C-EUC1206
- C15: device rcl:C-EUC0805 -> rcl:R-EU_R0603
- R3, R4: device rcl:R-EU_M0805 -> rcl:R-EU_R0603
Connections:
- net GND: now also C25.2
- net VCC: now also C25.1
Other:
- moved on the sheet: C15
Changed lines of the file:
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@@
 <part name="GND5" library="supply1" library_urn="urn:adsk.eagle:library:371" deviceset="GND" device=""/>
 <part name="C14" library="eagle-ltspice" library_urn="urn:adsk.eagle:library:217" deviceset="C" device="C0603" package3d_urn="urn:adsk.eagle:package:13262/1" value="100n"/>
-<part name="C12" library="rcl" library_urn="urn:adsk.eagle:library:334" deviceset="C-EU" device="C0805" package3d_urn="urn:adsk.eagle:package:23617/2" value="100n"/>
+<part name="C12" library="rcl" library_urn="urn:adsk.eagle:library:334" deviceset="C-EU" device="C0603" package3d_urn="urn:adsk.eagle:package:23616/2" value="100n"/>
 <part name="C9" library="eagle-ltspice" library_urn="urn:adsk.eagle:library:217" deviceset="C" device="C0603" package3d_urn="urn:adsk.eagle:package:13262/1" value="100n"/>
 <part name="C8" library="eagle-ltspice" library_urn="urn:adsk.eagle:library:217" deviceset="C" device="C0603" package3d_urn="urn:adsk.eagle:package:13262/1" value="100n"/>
@@
 <part name="SUPPLY2" library="supply2" library_urn="urn:adsk.eagle:library:372" deviceset="VCC" device=""/>
 <part name="C3" library="eagle-ltspice" library_urn="urn:adsk.eagle:library:217" deviceset="C" device="C0603" package3d_urn="urn:adsk.eagle:package:13262/1" value="10u"/>
-<part name="C1" library="rcl" library_urn="urn:adsk.eagle:library:334" deviceset="C-EU" device="C0805" package3d_urn="urn:adsk.eagle:package:23617/2" value="100n"/>
-<part name="C13" library="rcl" library_urn="urn:adsk.eagle:library:334" deviceset="C-EU" device="C0805" package3d_urn="urn:adsk.eagle:package:23617/2" value="10uF"/>
-<part name="C15" library="rcl" library_urn="urn:adsk.eagle:library:334" deviceset="C-EU" device="C0805" package3d_urn="urn:adsk.eagle:package:23617/2" value="100n"/>
+<part name="C1" library="rcl" library_urn="urn:adsk.eagle:library:334" deviceset="C-EU" device="C1206" package3d_urn="urn:adsk.eagle:package:23618/2" value="100nF"/>
+<part name="C13" library="rcl" library_urn="urn:adsk.eagle:library:334" deviceset="C-EU" device="C1206" package3d_urn="urn:adsk.eagle:package:23618/2" value="10uF"/>
+<part name="C15" library="rcl" library_urn="urn:adsk.eagle:library:334" deviceset="R-EU_" device="R0603" package3d_urn="urn:adsk.eagle:package:23555/3" value="100n"/>
 <part name="LED2" library="led" library_urn="urn:adsk.eagle:library:259" deviceset="LED" device="SML0805" package3d_urn="urn:adsk.eagle:package:15830/1" value="LED"/>
 <part name="PWR" library="led" library_urn="urn:adsk.eagle:library:259" deviceset="LED" device="SML0805" package3d_urn="urn:adsk.eagle:package:15830/1" value="LED"/>
-<part name="R3" library="rcl" library_urn="urn:adsk.eagle:library:334" deviceset="R-EU_" device="M0805" package3d_urn="urn:adsk.eagle:package:23556/2" value="10k"/>
+<part name="R3" library="rcl" library_urn="urn:adsk.eagle:library:334" deviceset="R-EU_" device="R0603" package3d_urn="urn:adsk.eagle:package:23555/3" value="10k"/>
 <part name="JP2" library="jumper" library_urn="urn:adsk.eagle:library:252" deviceset="JP3Q" device="" package3d_urn="urn:adsk.eagle:package:15460/1"/>
 <part name="JTAG" library="microbuilder" deviceset="HEADER-1X6" device="ROUND" value="JTAG"/>
 <part name="IC2" library="terriblefire" deviceset="XC9572XL-VQ64" device=""/>
 <part name="R1" library="rcl" library_urn="urn:adsk.eagle:library:334" deviceset="R-EU_" device="M1206" package3d_urn="urn:adsk.eagle:package:23566/2" value="4K7"/>
-<part name="R4" library="rcl" library_urn="urn:adsk.eagle:library:334" deviceset="R-EU_" device="M0805" package3d_urn="urn:adsk.eagle:package:23556/2" value="10k"/>
+<part name="R4" library="rcl" library_urn="urn:adsk.eagle:library:334" deviceset="R-EU_" device="R0603" package3d_urn="urn:adsk.eagle:package:23555/3" value="10k"/>
 <part name="SUPPLY10" library="supply2" library_urn="urn:adsk.eagle:library:372" deviceset="VCC" device=""/>
 <part name="D1" library="diode" library_urn="urn:adsk.eagle:library:210" deviceset="BAT54" device="" package3d_urn="urn:adsk.eagle:package:43389/2"/>
@@
 <part name="R6" library="rcl" library_urn="urn:adsk.eagle:library:334" deviceset="R-EU_" device="M0805" package3d_urn="urn:adsk.eagle:package:23556/2" value="100K"/>
 <part name="R7" library="rcl" library_urn="urn:adsk.eagle:library:334" deviceset="R-EU_" device="M0805" package3d_urn="urn:adsk.eagle:package:23556/2" value="100K"/>
+<part name="C25" library="rcl" library_urn="urn:adsk.eagle:library:334" deviceset="C-EU" device="C0603" package3d_urn="urn:adsk.eagle:package:23616/2" value="100n"/>
 </parts>
 <sheets>
@@
 <attribute name="NAME" x="1.27" y="270.2814" size="1.778" layer="95" rot="R180"/>
 <attribute name="VALUE" x="1.27" y="275.082" size="1.778" layer="96" rot="R180"/>
+</instance>
+<instance part="C25" gate="G$1" x="109.22" y="299.72" smashed="yes">
+<attribute name="NAME" x="110.744" y="300.101" size="1.778" layer="95"/>
+<attribute name="VALUE" x="110.744" y="295.021" size="1.778" layer="96"/>
 </instance>
 </instances>
@@
 <junction x="86.36" y="218.44"/>
 <pinref part="C15" gate="G$1" pin="2"/>
-<wire x1="96.52" y1="223.52" x2="96.52" y2="218.44" width="0.1524" layer="91"/>
+<wire x1="101.6" y1="228.6" x2="96.52" y2="218.44" width="0.1524" layer="91"/>
 <pinref part="PWR" gate="G$1" pin="C"/>
 <wire x1="96.52" y1="218.44" x2="109.22" y2="218.44" width="0.1524" layer="91"/>
@@
 <junction x="-20.32" y="279.4"/>
 <label x="-25.4" y="289.56" size="1.778" layer="95"/>
+</segment>
+<segment>
+<pinref part="C25" gate="G$1" pin="2"/>
+<wire x1="109.22" y1="294.64" x2="109.22" y2="292.1" width="0.1524" layer="91"/>
+<wire x1="109.22" y1="292.1" x2="132.08" y2="292.1" width="0.1524" layer="91"/>
 </segment>
 </net>
@@
 <junction x="86.36" y="233.68"/>
 <pinref part="C15" gate="G$1" pin="1"/>
-<wire x1="96.52" y1="233.68" x2="96.52" y2="231.14" width="0.1524" layer="91"/>
+<wire x1="96.52" y1="233.68" x2="91.44" y2="228.6" width="0.1524" layer="91"/>
 <wire x1="96.52" y1="233.68" x2="104.14" y2="233.68" width="0.1524" layer="91"/>
 <junction x="96.52" y="233.68"/>
@@
 <label x="104.14" y="287.02" size="1.778" layer="95"/>
 </segment>
-</net>
+<segment>
+<pinref part="C25" gate="G$1" pin="1"/>
+<wire x1="109.22" y1="302.26" x2="109.22" y2="309.88" width="0.1524" layer="91"/>
+</segment>
+</net>

Commit message: updated footprint of 32Khz crystal
Parts:
- X1: value SMD-CRYSTAL-8MHZ-20PF-20PPM(2P-5.0X3.2MM) -> SMD-CRYSTAL-25MHZ-20PF-20PPM(2P-5.0X3.2MM)
- X2: value SMD-CRYSTAL-32768KHZ-20PF-20PPM(2P-5.0X3.2MM) -> 32.768KHZ; device SMD-CRYSTAL-8MHZ-20PF-20PPM_2P-5.0X3.2MM_:SMD-CRYSTAL-8MHZ-20PF-20PPM(2P-5.0X3.2MM) -> adafruit:XTAL-3.2X1.5
Connections:
- net LSE_OSCIN: now also X2.P$2; no longer X2.2
- net LSE_OSCOUT: now also X2.P$1; no longer X2.1
Other:
- moved on the sheet: C15
Changed lines of the file:
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@@
 <part name="G1" library="battery" library_urn="urn:adsk.eagle:library:109" deviceset="CH23-1220LF" device="" package3d_urn="urn:adsk.eagle:package:4614/1"/>
 <part name="U$1" library="board" deviceset="USB-A-2_USB_USB-A-2" device=""/>
-<part name="X1" library="SMD-CRYSTAL-8MHZ-20PF-20PPM_2P-5.0X3.2MM_" deviceset="SMD-CRYSTAL-8MHZ-20PF-20PPM(2P-5.0X3.2MM)" device=""/>
+<part name="X1" library="SMD-CRYSTAL-8MHZ-20PF-20PPM_2P-5.0X3.2MM_" deviceset="SMD-CRYSTAL-8MHZ-20PF-20PPM(2P-5.0X3.2MM)" device="" value="SMD-CRYSTAL-25MHZ-20PF-20PPM(2P-5.0X3.2MM)"/>
 <part name="JP1" library="SparkFun-Retired" deviceset="JUMPER-2" device="PTH"/>
 <part name="F1" library="eagle-ltspice" library_urn="urn:adsk.eagle:library:217" deviceset="R" device="R1206" package3d_urn="urn:adsk.eagle:package:13301/1" value="0R"/>
@@
 <part name="C24" library="eagle-ltspice" library_urn="urn:adsk.eagle:library:217" deviceset="C" device="C0603" package3d_urn="urn:adsk.eagle:package:13262/1" value="22p"/>
 <part name="GND1" library="supply1" library_urn="urn:adsk.eagle:library:371" deviceset="GND" device=""/>
-<part name="X2" library="SMD-CRYSTAL-8MHZ-20PF-20PPM_2P-5.0X3.2MM_" deviceset="SMD-CRYSTAL-8MHZ-20PF-20PPM(2P-5.0X3.2MM)" device="" value="SMD-CRYSTAL-32768KHZ-20PF-20PPM(2P-5.0X3.2MM)"/>
 <part name="JP3" library="SparkFun-Retired" deviceset="JUMPER-2" device="PTH"/>
 <part name="IC4" library="THS7314D" deviceset="THS7314D" device=""/>
@@
 <part name="R7" library="rcl" library_urn="urn:adsk.eagle:library:334" deviceset="R-EU_" device="M0805" package3d_urn="urn:adsk.eagle:package:23556/2" value="100K"/>
 <part name="C25" library="rcl" library_urn="urn:adsk.eagle:library:334" deviceset="C-EU" device="C0603" package3d_urn="urn:adsk.eagle:package:23616/2" value="100n"/>
+<part name="X2" library="adafruit" library_urn="urn:adsk.eagle:library:420" deviceset="XTAL" device="-3.2X1.5" package3d_urn="urn:adsk.eagle:package:6240808/1" value="32.768KHZ"/>
 </parts>
 <sheets>
@@
 <attribute name="VALUE" x="87.884" y="223.901" size="1.778" layer="96"/>
 </instance>
-<instance part="C15" gate="G$1" x="96.52" y="228.6" smashed="yes">
-<attribute name="NAME" x="98.044" y="228.981" size="1.778" layer="95"/>
-<attribute name="VALUE" x="98.044" y="223.901" size="1.778" layer="96"/>
+<instance part="C15" gate="G$1" x="96.52" y="226.06" smashed="yes" rot="R270">
+<attribute name="NAME" x="99.441" y="221.996" size="1.778" layer="95" rot="R270"/>
+<attribute name="VALUE" x="99.441" y="229.616" size="1.778" layer="96" rot="R270"/>
 </instance>
 <instance part="LED2" gate="G$1" x="22.86" y="76.2" smashed="yes" rot="R270">
@@
 <attribute name="VALUE" x="172.72" y="48.26" size="1.778" layer="96" rot="R90"/>
 </instance>
-<instance part="X2" gate="G$1" x="147.32" y="50.8" smashed="yes" rot="R90">
-<attribute name="NAME" x="144.77693125" y="48.25693125" size="1.27153125" layer="95" ratio="10" rot="R90"/>
-</instance>
 <instance part="JP3" gate="A" x="147.32" y="248.92" smashed="yes" rot="R270">
 <attribute name="NAME" x="147.32" y="250.19" size="1.778" layer="95"/>
@@
 <attribute name="VALUE" x="110.744" y="295.021" size="1.778" layer="96"/>
 </instance>
+<instance part="X2" gate="G$1" x="147.32" y="50.8" smashed="yes" rot="R90">
+<attribute name="NAME" x="143.51" y="48.26" size="1.27" layer="95" font="vector" rot="R90"/>
+<attribute name="VALUE" x="152.4" y="46.99" size="1.27" layer="96" font="vector" rot="R90"/>
+</instance>
 </instances>
 <busses>
@@
 <junction x="86.36" y="218.44"/>
 <pinref part="C15" gate="G$1" pin="2"/>
-<wire x1="101.6" y1="228.6" x2="96.52" y2="218.44" width="0.1524" layer="91"/>
+<wire x1="96.52" y1="220.98" x2="96.52" y2="218.44" width="0.1524" layer="91"/>
 <pinref part="PWR" gate="G$1" pin="C"/>
 <wire x1="96.52" y1="218.44" x2="109.22" y2="218.44" width="0.1524" layer="91"/>
@@
 <junction x="86.36" y="233.68"/>
 <pinref part="C15" gate="G$1" pin="1"/>
-<wire x1="96.52" y1="233.68" x2="91.44" y2="228.6" width="0.1524" layer="91"/>
+<wire x1="96.52" y1="233.68" x2="96.52" y2="231.14" width="0.1524" layer="91"/>
 <wire x1="96.52" y1="233.68" x2="104.14" y2="233.68" width="0.1524" layer="91"/>
 <junction x="96.52" y="233.68"/>
@@
 <wire x1="154.94" y1="55.88" x2="147.32" y2="55.88" width="0.1524" layer="91"/>
 <pinref part="C23" gate="G$1" pin="1"/>
-<pinref part="X2" gate="G$1" pin="2"/>
 <wire x1="147.32" y1="55.88" x2="147.32" y2="54.61" width="0.1524" layer="91"/>
 <label x="134.62" y="60.96" size="1.778" layer="95"/>
 <wire x1="147.32" y1="55.88" x2="132.08" y2="55.88" width="0.1524" layer="91"/>
 <junction x="147.32" y="55.88"/>
+<pinref part="X2" gate="G$1" pin="P$2"/>
 </segment>
 <segment>
@@
 <wire x1="154.94" y1="45.72" x2="147.32" y2="45.72" width="0.1524" layer="91"/>
 <pinref part="C24" gate="G$1" pin="1"/>
-<pinref part="X2" gate="G$1" pin="1"/>
 <wire x1="147.32" y1="45.72" x2="147.32" y2="46.99" width="0.1524" layer="91"/>
 <wire x1="147.32" y1="45.72" x2="132.08" y2="45.72" width="0.1524" layer="91"/>
 <junction x="147.32" y="45.72"/>
 <label x="134.62" y="43.18" size="1.778" layer="95"/>
+<pinref part="X2" gate="G$1" pin="P$1"/>
 </segment>
 <segment>
